File: LMR16006-Breakout.kicad_pcb (KiCad board)
At the start: 2 copper layers, 21 x 21 mm, 16 parts, among them P1 CONN_01X04, U1 LMR16006

Commit message: silkscreen description, oshw logo
Parts:
- added REF***: OSHW-Logo_7.5x8mm_SilkScreen, Symbols:OSHW-Logo_7.5x8mm_SilkScreen, B.Cu at (130.2, 94.8)
Other:
- board text added: "LMR16006 60V Buck converter 0,6A V1"
- board text added: "by Florian Winkler"

Commit message: labels for pinheader
Other:
- board text added: "GND"
- board text added: "SHDN"
- board text added: "VCC"
- board text added: "Vout"
Changed lines of the file:
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@@
     (area 119.924999 88.924999 141.075001 110.075001)
     (thickness 1.6)
-    (drawings 11)
+    (drawings 15)
     (tracks 154)
     (zones 0)
@@
       (xy 0.500964 3.601424)) (layer B.SilkS) (width 0.01))
   )
-  (gr_text "LMR16006\n60V Buck converter\n0,6A\nV1" (at 139.05 104.92) (layer B.SilkS)
+  (gr_text Vout (at 133.97 106.825 90) (layer B.SilkS)
+    (effects (font (size 1 1) (thickness 0.2)) (justify right mirror))
+  )
+  (gr_text GND (at 131.43 106.825 90) (layer B.SilkS)
+    (effects (font (size 1 1) (thickness 0.2)) (justify right mirror))
+  )
+  (gr_text SHDN (at 128.89 106.825 90) (layer B.SilkS)
+    (effects (font (size 1 1) (thickness 0.2)) (justify right mirror))
+  )
+  (gr_text VCC (at 126.35 106.825 90) (layer B.SilkS)
+    (effects (font (size 1 1) (thickness 0.2)) (justify right mirror))
+  )
+  (gr_text "LMR16006\n60V Buck converter\n0,6A\nV1" (at 137.145 95.395 90) (layer B.SilkS)
     (effects (font (size 0.8 0.8) (thickness 0.1)) (justify left mirror))
   )
